File: esp32-crystal-ball.kicad_sch (KiCad schematic)
At the start: 52 parts, among them J1 TYPE-C-31-M-12, J2 Barrel_Jack_Switch, J3 Screw_Terminal_01x03, J4 Conn_02x03_Counter_Clockwise, J5 Conn_01x02_Pin, Q1 NTA4151PT1G, U1 ESP32-S3-MINI-1, U2 OWMMOD-403010A-S261F, U3 NCP167BMX330TBG, U4 SN74LV1T34DBV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

Commit message: Adds images and README file.
Parts:
- QWIIC2: now fitted; now in the parts list
Connections:
- net LED_DIN: no longer D3.2 (DIN), TP1.1, U4.4 (Y)
- new net: D3.2 (DIN), TP1.1, U4.4 (Y)
Other:
- note added: "Link to power LEDs directly or from barrel jack"
- moved on the sheet: C8, TP1, TP5, U4

Commit message: Fixes voltage regulator footprint
Parts:
- removed BOOT1, EN1: B3U-3000P, B3U-3000P:SW_B3U-3000P, symbol B3U-3000P:B3U-3000P
- added SW1, SW2: TS24CA, easyeda2kicad:SW-SMD_TS24CA, symbol EasyEDA2Kicad:TS24CA
- U3: footprint NCP167BMX330TBG:VREG_NCP167BMX330TBG -> NCP167BMX330TBG-v2:VREG_NCP167BMX330TBG
Connections:
- net BOOT: now also SW1.4
- net EN: now also SW2.4
- net GND: now also SW1.1, SW1.22 (2), SW1.3, SW2.1, SW2.22 (2), SW2.3
